File: pcb/dev_board.kicad_sch (KiCad schematic)
At the start: 29 parts, among them J1 Conn_02x13_Odd_Even, J2 Conn_02x13_Odd_Even, SW1 SW_DIP_x03, SW2 ARM, U1 LPC, U2 MCP3202, U3 TLV74325, U4 TLV74318, U5 LPC, U6 TLV74318

Commit message: V0.1 schematic complete, pcb placed. emulator connections, 24-stqfn LPC fanout in place.
Parts:
- removed C2: 4.7u, Capacitor_SMD:C_1206_3216Metric, symbol Device:C_Small
- removed U3: TLV74325, Package_TO_SOT_SMD:SOT-23-5, symbol myspace:TLV74325_SOT23-5
- removed U4: TLV74318, Package_TO_SOT_SMD:SOT-23-5, symbol myspace:TLV74325_SOT23-5
- removed U5: LPC, myspace pcb:QFN-24-3x3mm, symbol myspace:SLG47910V
- added D6: DT1042-04SO-7, Package_TO_SOT_SMD:SOT-23-6, symbol Power_Protection:DT1240A-08LP3810
- added J4: Conn_01x05, Connector_PinHeader_2.54mm:PinHeader_1x05_P2.54mm_Vertical_SMD_Pin1Left, symbol Connector_Generic:Conn_01x05
- added R11, R12, R13, R14, R16: 47, Resistor_SMD:R_0603_1608Metric, symbol Device:R
- added R15: 1R 3W 0.1%, Resistor_SMD:R_2512_6332Metric, symbol Device:R
- added R6: 1K, Resistor_SMD:R_0603_1608Metric, symbol Device:R
- added R7: 1K5, Resistor_SMD:R_0603_1608Metric, symbol Device:R
- added R8: 18R6, Resistor_SMD:R_0603_1608Metric, symbol Device:R
- added R9: 3k3, Resistor_SMD:R_0603_1608Metric, symbol Device:R
- added U3: TLV75530PDBV, Package_TO_SOT_SMD:SOT-23-5, symbol Regulator_Linear:TLV75530PDBV
- C3: value 4.7u -> 22n; footprint Capacitor_SMD:C_1206_3216Metric -> Capacitor_SMD:C_0603_1608Metric; DPN 399-C1206C475K5PAC7800CT-ND -> 399-C0603C105K3RAC7867CT-ND
- C5, C6: value 1u -> 22n
- R1: value 10K -> 0R; DPN 311-10.0KHRCT-ND -> P0.0GCT-ND; JLC C778416 -> C491211
- R10: renamed from RV1; value R_Potentiometer_US -> 1K5
- R5: value 10K -> DNI; DPN 311-10.0KHRCT-ND -> (none); JLC C778416 -> C491211
- U1: value LPC -> XS-LPC-01
- U6: value TLV74318 -> TLV74311
Connections:
- net +2V5 is gone; now on net +3V0: C7.1
- net arm_led is gone; now on net adc_ncs: J2.25 (Pin_25), U1.9 (GPIO18)
- net charge is gone; now on net run_led: J1.6 (Pin_6), U1.20 (GPIO7)
- net cont_led is gone; now on net setup: J2.5 (Pin_5), U1.23 (GPIO8)
- net cs is gone; now on net adc_miso: J2.21 (Pin_21), U1.7 (GPIO16)
- net dataA0 is gone; now on net time_led: J2.13 (Pin_13), U1.3 (GPIO12)
- net dataB1 is gone; now on net adc_clk: J2.19 (Pin_19), U1.6 (GPIO15)
- net dump is gone; now on net period: J2.9 (Pin_9), U1.1 (GPIO10)
- net launch_n is gone; now on net fault_led: J2.7 (Pin_7), U1.24 (GPIO9)
- net pwm is gone; now on net adc_mosi: J2.23 (Pin_23), U1.8 (GPIO17)
- net sclk is gone; now on net timeout: J2.11 (Pin_11), U1.2 (GPIO11)
- net speaker is gone; now on net start: J1.20 (Pin_20), U1.13 (GPIO0)
- net +1V1: no longer C6.1
- net +3.3V: now also U6.3 (EN), D6.5 (vdd), J4.1 (Pin_1), R9.2, U3.1 (IN), U3.3 (EN); no longer C1.1, C3.1, C5.1, R1.1, R5.1
- net GND: now also R2.2, R3.2, R4.2, R5.1, SW2.1, U2.4 (VSS), D6.2 (vss), J4.3 (Pin_3), R7.2, U3.2 (GND)
- net reset_n: now also R1.2, R5.2; no longer J1.24 (Pin_24)
- net spi_ss: now also R9.1
- net run_led: now reaches D1.2 (A)
- net +3V0: now reaches R10.1
- net +3V0: now also U2.8 (VDD/VREF), U3.5 (OUT)
- net at R10.2: now also R12.1
- net CT2: now reaches R10.3
- net CT2: now also C1.1, C3.1, J4.5 (Pin_5), R15.2, R16.2, R7.1, R8.2
- net fault_led: now reaches D2.2 (A)
- net start: now reaches SW2.2
- net time_led: now reaches D3.2 (A)
- net adc_ncs: now reaches U2.1 (~{CS}/SHDN)
- net at U2.2 (CH0): now also C6.1, R11.2
- net at U2.3 (CH1): now also C5.1, R12.2
- net adc_mosi: now reaches U2.5 (DIN)
- net adc_miso: now reaches U2.6 (DOUT)
- net adc_clk: now reaches U2.7 (CLK)
- net timeout: now reaches SW1.4
- net period: now reaches SW1.5
- net setup: now reaches SW1.6
- net dataA1: no longer names the net of J2.17 (Pin_17), U1.5 (GPIO14)
- net dataB0: no longer names the net of J2.15 (Pin_15), U1.4 (GPIO13)
- net mute_n renamed pump
- net pump: now also R13.2, R6.1
- new net: D6.4 (K1), R13.1
- new net: D6.1 (X1), R16.1
- new net: D6.6 (K2), R14.1
- new net: J1.24 (Pin_24), R1.1
- new net CT1: J4.4 (Pin_4), R11.1, R14.2, R15.1, R8.1
- new net out: J4.2 (Pin_2), R6.2
- no-connect marks 1 -> 2
Other:
- note added: "Analog to Digital"
- note added: "Connector"
- note added: "FRONT PANEL"
- note added: "LPC Pump Controller"
- note removed: "ALT XS"
- note removed: "Evaluation Probe"
- note removed: "LPC Dev Board"
- note removed: "Liquid Pump Controller"
- note removed: "XS LPC"
- moved on the sheet: C10, C4, C7, C8, C9, D1, D2, D3, J1, J2, R10, R2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

Commit message: Update BOM to v0.1 with in-stock, current Digikey Parts Numbers
Parts:
- C3, C5, C6: DPN 399-C0603C105K3RAC7867CT-ND -> 445-5663-1-ND
- D6: DPN (none) -> DT1042-04SO-7DICT-ND
- J4: DPN (none) -> SAM10797-ND
- R10: value 1K5 -> 1K; DPN (none) -> SM-42TW102CT-ND
- R11, R12, R13, R14, R16: DPN 311-10.0KHRCT-ND -> 541-47.0HCT-ND
- R15: DPN 311-10.0KHRCT-ND -> 738-RNCL2512FT1R00CT-ND
- R2, R3, R4, R6: DPN P1.00KHCT-ND -> 541-1.00KHCT-ND
- R7: value 1K5 -> 1K; DPN 311-10.0KHRCT-ND -> 541-1.00KHCT-ND
- R8: DPN 311-10.0KHRCT-ND -> 311-18.2HRCT-ND
- SW1: DPN CT2193LPST-ND -> 563-CFS-0300TACT-ND
- SW2: value ARM -> Start
- U2: DPN (none) -> MCP3202-CI/MS-ND
- U3: DPN (none) -> 576-4905-1-ND
- U6: DPN 296-48712-1-ND -> 296-50002-1-ND
Other:
- title: XS-LPCDB Development Board -> XS-LPC-DB Development Board
