File: pcb/dev_board.kicad_sch (KiCad schematic)
At the start: 37 parts, among them J1 Conn_02x13_Odd_Even, J2 Conn_02x13_Odd_Even, J4 Conn_01x05, SW1 SW_DIP_x03, SW2 Start, U1 XS-LPC-01, U2 MCP3202, U3 NCP114ASN280T1G, U6 TLV74311

Commit message: v0.3 emulator winged, clean routed PCB, schem, Digikey BOM. For review and cleanup.
Parts:
- removed C7: 1u, Capacitor_SMD:C_0603_1608Metric, symbol Device:C_Small
- added C11: 0.1u, Capacitor_SMD:C_0603_1608Metric, symbol Device:C_Small
- added C12: 10u, Capacitor_SMD:C_1206_3216Metric, symbol Device:C_Small
- added C2: 1u, Capacitor_SMD:C_0603_1608Metric, symbol Device:C_Small
Connections:
- net +3.3V: now also C2.1
- net +3V0: now also C11.1, C12.1
- net GND: now also C11.2, C12.2, C2.2
- net fault_led: now also J2.13 (Pin_13), U1.3 (GPIO12); no longer J2.7 (Pin_7), U1.24 (GPIO9)
- net period: now also J2.5 (Pin_5), U1.23 (GPIO8); no longer J2.9 (Pin_9), U1.1 (GPIO10)
- net pump: now also J2.7 (Pin_7), U1.24 (GPIO9); no longer J1.18 (Pin_18), U1.14 (GPIO1)
- net run_led: now also J2.15 (Pin_15), U1.4 (GPIO13); no longer J1.6 (Pin_6), U1.20 (GPIO7)
- net setup: now also J1.6 (Pin_6), U1.20 (GPIO7); no longer J2.5 (Pin_5), U1.23 (GPIO8)
- net time_led: now also J2.11 (Pin_11), U1.2 (GPIO11); no longer J2.13 (Pin_13), U1.3 (GPIO12)
- net timeout: now also J2.9 (Pin_9), U1.1 (GPIO10); no longer J2.11 (Pin_11), U1.2 (GPIO11)
- new net: J1.18 (Pin_18), U1.14 (GPIO1)
Other:
- moved on the sheet: C8
