File: pcb/dev_board.kicad_sch (KiCad schematic)
At the start: 40 parts, among them J1 Conn_02x13_Odd_Even, J2 Conn_02x13_Odd_Even, J4 Conn_01x05, SW1 SW_DIP_x03, SW2 Start, U1 XS-LPC-01, U2 MCP3202, U3 NCP114ASN280T1G, U6 TLV74311

Commit message: Update DB pcb and sch files to 0.5.1 to reflect swapped run/tile LEDs with correct net names. No change to PCB
Parts:
- renumbered D3 to D1, D1 to D3, R4 to R2, R2 to R4
Connections:
- net run_led: now also J2.11 (Pin_11), U1.2 (GPIO11); no longer J2.15 (Pin_15), U1.4 (GPIO13)
- net time_led: now also J2.15 (Pin_15), U1.4 (GPIO13); no longer J2.11 (Pin_11), U1.2 (GPIO11)
