File: pcb/dev_board.kicad_pcb (KiCad board)
At the start: 6 copper layers, 45.7 x 42.2 mm, 40 parts, among them J1 Conn_02x13_Odd_Even, J2 Conn_02x13_Odd_Even, J4 Conn_01x05, SW1 SW_DIP_x03, SW2 Start, U1 XS-LPC-01, U2 MCP3202, U3 NCP114ASN280T1G, U6 TLV74311

Commit message: Update DB pcb and sch files to 0.5.1 to reflect swapped run/tile LEDs with correct net names. No change to PCB
Parts:
- D1: value RUN -> TME
- D3: value TME -> RUN
Connections:
- D1 pad 2: /run_led -> /time_led
- D3 pad 2: /time_led -> /run_led
- J2 pad 11: /time_led -> /run_led
- J2 pad 15: /run_led -> /time_led
- U1 pad 2: /time_led -> /run_led
- U1 pad 4: /run_led -> /time_led
Routing:
- net /time_led: track 44.4 -> 39.6 mm
- net /run_led: track 39.6 -> 44.4 mm
Changed lines of the file:
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@@
     (title "XS-LPC-DB Development Board")
     (date "2026-07-10")
-    (rev "v0.5")
+    (rev "v0.5.1")
     (company "Eric Pearson: XYZZY Semiconductor")
   )
@@
         (effects (font (size 1 1) (thickness 0.15)))
     )
-    (fp_text value "RUN" (at 0 1.43) (layer "F.Fab")
+    (fp_text value "TME" (at 0 1.43) (layer "F.Fab")
         (effects (font (size 1 1) (thickness 0.15)))
     )
@@
       (net 12 "Net-(D1-K)") (pinfunction "K") (pintype "passive"))
     (pad "2" smd roundrect (at 0.7875 0 180) (size 0.875 0.95) (layers "F.Cu" "F.Paste" "F.Mask") (roundrect_rratio 0.25)
-      (net 18 "/run_led") (pinfunction "A") (pintype "passive"))
+      (net 20 "/time_led") (pinfunction "A") (pintype "passive"))
     (model "${KICAD6_3DMODEL_DIR}/LED_SMD.3dshapes/LED_0603_1608Metric.wrl"
       (offset (xyz 0 0 0))
@@
         (effects (font (size 1 1) (thickness 0.15)))
     )
-    (fp_text value "TME" (at 0 1.43) (layer "F.Fab")
+    (fp_text value "RUN" (at 0 1.43) (layer "F.Fab")
         (effects (font (size 1 1) (thickness 0.15)))
     )
@@
       (net 10 "Net-(D3-K)") (pinfunction "K") (pintype "passive"))
     (pad "2" smd roundrect (at 0.7875 0 180) (size 0.875 0.95) (layers "F.Cu" "F.Paste" "F.Mask") (roundrect_rratio 0.25)
-      (net 20 "/time_led") (pinfunction "A") (pintype "passive"))
+      (net 18 "/run_led") (pinfunction "A") (pintype "passive"))
     (model "${KICAD6_3DMODEL_DIR}/LED_SMD.3dshapes/LED_0603_1608Metric.wrl"
       (offset (xyz 0 0 0))
@@
       ))
     (pad "2" smd roundrect (at -1.5 -0.6) (size 0.75 0.2) (layers "F.Cu" "F.Paste" "F.Mask") (roundrect_rratio 0.25)
-      (net 20 "/time_led") (pinfunction "GPIO11") (pintype "bidirectional"))
+      (net 18 "/run_led") (pinfunction "GPIO11") (pintype "bidirectional"))
     (pad "3" smd roundrect (at -1.5 -0.2) (size 0.75 0.2) (layers "F.Cu" "F.Paste" "F.Mask") (roundrect_rratio 0.25)
       (net 19 "/fault_led") (pinfunction "GPIO12") (pintype "bidirectional"))
     (pad "4" smd roundrect (at -1.5 0.2) (size 0.75 0.2) (layers "F.Cu" "F.Paste" "F.Mask") (roundrect_rratio 0.25)
-      (net 18 "/run_led") (pinfunction "GPIO13") (pintype "bidirectional"))
+      (net 20 "/time_led") (pinfunction "GPIO13") (pintype "bidirectional"))
     (pad "5" smd roundrect (at -1.5 0.6) (size 0.75 0.2) (layers "F.Cu" "F.Paste" "F.Mask") (roundrect_rratio 0.25)
       (net 25 "Net-(J2-Pin_17)") (pinfunction "GPIO14") (pintype "bidirectional"))
@@
       (net 11 "GND") (pinfunction "Pin_10") (pintype "passive"))
     (pad "11" thru_hole oval (at 0 -12.7 180) (size 1.7 1.7) (drill 1) (layers "*.Cu" "*.Mask")
-      (net 20 "/time_led") (pinfunction "Pin_11") (pintype "passive"))
+      (net 18 "/run_led") (pinfunction "Pin_11") (pintype "passive"))
     (pad "12" thru_hole oval (at -2.54 -12.7 180) (size 1.7 1.7) (drill 1) (layers "*.Cu" "*.Mask")
       (net 11 "GND") (pinfunction "Pin_12") (pintype "passive"))
@@
       (net 11 "GND") (pinfunction "Pin_14") (pintype "passive"))
     (pad "15" thru_hole oval (at 0 -17.78 180) (size 1.7 1.7) (drill 1) (layers "*.Cu" "*.Mask")
-      (net 18 "/run_led") (pinfunction "Pin_15") (pintype "passive"))
+      (net 20 "/time_led") (pinfunction "Pin_15") (pintype "passive"))
     (pad "16" thru_hole oval (at -2.54 -17.78 180) (size 1.7 1.7) (drill 1) (layers "*.Cu" "*.Mask")
       (net 11 "GND") (pinfunction "Pin_16") (pintype "passive"))
@@
   (gr_line (start 177.292 121.92) (end 177.292 86.4108)
     (stroke (width 0.15) (type default)) (layer "B.SilkS"))
-  (gr_rect (start 181.258 108.0796) (end 182.978 106.0196)
+  (gr_rect (start 181.258 106.0196) (end 182.978 108.0796)
     (stroke (width 0.15) (type default)) (fill none) (layer "F.SilkS"))
   (gr_line (start 163.068 121.92) (end 163.068 86.36)
@@
   (segment (start 168.275 112.255) (end 168.45 112.08) (width 0.254) (layer "B.Cu") (net 17))
   (segment (start 170.3125 112.08) (end 168.45 112.08) (width 0.254) (layer "B.Cu") (net 17))
-  (segment (start 165.604 105.3515) (end 166.013 104.9425) (width 0.254) (layer "F.Cu") (net 18))
-  (segment (start 166.013 104.9425) (end 168.604 104.9425) (width 0.254) (layer "F.Cu") (net 18))
-  (segment (start 165.3765 86.2489) (end 164.2364 87.389) (width 0.254) (layer "F.Cu") (net 18))
-  (segment (start 164.2364 87.389) (end 164.2364 103.9839) (width 0.254) (layer "F.Cu") (net 18))
-  (segment (start 164.2364 103.9839) (end 165.604 105.3515) (width 0.254) (layer "F.Cu") (net 18))
-  (via (at 165.604 105.3515) (size 0.6) (drill 0.35) (layers "F.Cu" "B.Cu") (net 18))
-  (segment (start 149.86 106.68) (end 151.0792 105.4608) (width 0.254) (layer "In2.Cu") (net 18))
-  (segment (start 165.4947 105.4608) (end 165.604 105.3515) (width 0.254) (layer "In2.Cu") (net 18))
-  (segment (start 151.0792 105.4608) (end 165.4947 105.4608) (width 0.254) (layer "In2.Cu") (net 18))
+  (segment (start 165.906 102.9359) (end 167.1088 104.1387) (width 0.254) (layer "F.Cu") (net 18))
+  (segment (start 172.819 86.9214) (end 172.212 87.5284) (width 0.254) (layer "F.Cu") (net 18))
+  (segment (start 165.5064 88.3412) (end 165.5064 102.5363) (width 0.254) (layer "F.Cu") (net 18))
+  (segment (start 166.3192 87.5284) (end 165.5064 88.3412) (width 0.254) (layer "F.Cu") (net 18))
+  (segment (start 165.5064 102.5363) (end 165.906 102.9359) (width 0.254) (layer "F.Cu") (net 18))
+  (segment (start 172.212 87.5284) (end 166.3192 87.5284) (width 0.254) (layer "F.Cu") (net 18))
+  (segment (start 167.1088 104.1387) (end 168.5758 104.1387) (width 0.254) (layer "F.Cu") (net 18))
+  (segment (start 172.819 86.0589) (end 172.819 86.9214) (width 0.254) (layer "F.Cu") (net 18))
+  (via (at 165.906 102.9359) (size 0.6) (drill 0.35) (layers "F.Cu" "B.Cu") (net 18))
+  (segment (start 151.13 100.33) (end 156.21 100.33) (width 0.254) (layer "In2.Cu") (net 18))
+  (segment (start 158.8516 102.9716) (end 165.8703 102.9716) (width 0.254) (layer "In2.Cu") (net 18))
+  (segment (start 149.86 101.6) (end 151.13 100.33) (width 0.254) (layer "In2.Cu") (net 18))
+  (segment (start 156.21 100.33) (end 158.8516 102.9716) (width 0.254) (layer "In2.Cu") (net 18))
+  (segment (start 165.8703 102.9716) (end 165.906 102.9359) (width 0.254) (layer "In2.Cu") (net 18))
   (segment (start 164.846 103.3999) (end 165.5758 104.1297) (width 0.254) (layer "F.Cu") (net 19))
   (segment (start 169.169 86.7614) (end 168.91 87.0204) (width 0.254) (layer "F.Cu") (net 19))
@@
   (segment (start 149.86 104.14) (end 151.13 102.87) (width 0.254) (layer "In2.Cu") (net 19))
   (segment (start 157.1196 102.87) (end 158.3793 104.1297) (width 0.254) (layer "In2.Cu") (net 19))
-  (segment (start 165.906 102.9359) (end 167.1088 104.1387) (width 0.254) (layer "F.Cu") (net 20))
-  (segment (start 172.819 86.9214) (end 172.212 87.5284) (width 0.254) (layer "F.Cu") (net 20))
-  (segment (start 165.5064 88.3412) (end 165.5064 102.5363) (width 0.254) (layer "F.Cu") (net 20))
-  (segment (start 166.3192 87.5284) (end 165.5064 88.3412) (width 0.254) (layer "F.Cu") (net 20))
-  (segment (start 165.5064 102.5363) (end 165.906 102.9359) (width 0.254) (layer "F.Cu") (net 20))
-  (segment (start 172.212 87.5284) (end 166.3192 87.5284) (width 0.254) (layer "F.Cu") (net 20))
-  (segment (start 167.1088 104.1387) (end 168.5758 104.1387) (width 0.254) (layer "F.Cu") (net 20))
-  (segment (start 172.819 86.0589) (end 172.819 86.9214) (width 0.254) (layer "F.Cu") (net 20))
-  (via (at 165.906 102.9359) (size 0.6) (drill 0.35) (layers "F.Cu" "B.Cu") (net 20))
-  (segment (start 151.13 100.33) (end 156.21 100.33) (width 0.254) (layer "In2.Cu") (net 20))
-  (segment (start 158.8516 102.9716) (end 165.8703 102.9716) (width 0.254) (layer "In2.Cu") (net 20))
-  (segment (start 149.86 101.6) (end 151.13 100.33) (width 0.254) (layer "In2.Cu") (net 20))
-  (segment (start 156.21 100.33) (end 158.8516 102.9716) (width 0.254) (layer "In2.Cu") (net 20))
-  (segment (start 165.8703 102.9716) (end 165.906 102.9359) (width 0.254) (layer "In2.Cu") (net 20))
+  (segment (start 165.604 105.3515) (end 166.013 104.9425) (width 0.254) (layer "F.Cu") (net 20))
+  (segment (start 166.013 104.9425) (end 168.604 104.9425) (width 0.254) (layer "F.Cu") (net 20))
+  (segment (start 165.3765 86.2489) (end 164.2364 87.389) (width 0.254) (layer "F.Cu") (net 20))
+  (segment (start 164.2364 87.389) (end 164.2364 103.9839) (width 0.254) (layer "F.Cu") (net 20))
+  (segment (start 164.2364 103.9839) (end 165.604 105.3515) (width 0.254) (layer "F.Cu") (net 20))
+  (via (at 165.604 105.3515) (size 0.6) (drill 0.35) (layers "F.Cu" "B.Cu") (net 20))
+  (segment (start 149.86 106.68) (end 151.0792 105.4608) (width 0.254) (layer "In2.Cu") (net 20))
+  (segment (start 165.4947 105.4608) (end 165.604 105.3515) (width 0.254) (layer "In2.Cu") (net 20))
+  (segment (start 151.0792 105.4608) (end 165.4947 105.4608) (width 0.254) (layer "In2.Cu") (net 20))
   (segment (start 165.807 118.2349) (end 167.95775 120.38565) (width 0.254) (layer "F.Cu") (net 21))
   (segment (start 172.0912 105.7423) (end 171.6212 105.7423) (width 0.254) (layer "F.Cu") (net 21))
@@
         (xy 179.07 96.52)
         (xy 176.3268 96.52)
-        (xy 176.3268 96.52)
-        (xy 163.83 96.52)
         (xy 163.83 96.52)
         (xy 161.29 96.52)
@@
         (xy 177.292 113.665)
         (xy 174.625 113.665)
-        (xy 174.625 113.665)
         (xy 168.275 113.665)
